File: pcb/v0/v0.kicad_pcb (KiCad board)
At the start: 4 copper layers, 100 x 100 mm, 23 parts, among them J1 Screw_Terminal_01x02, J2 Screw_Terminal_01x02, J3 Conn_01x08, J6 RAM, SW1 SW_DIP_x04

Commit message: substrate fixes
Parts:
- added R6: 470, Resistor_SMD:R_0402_1005Metric, F.Cu at (109.2, 21.9)
- added TP1: TestPoint, TestPoint:TestPoint_Pad_D1.0mm, B.Cu at (48.2, 23.9)
- added TP10: TestPoint, TestPoint:TestPoint_Pad_D1.0mm, B.Cu at (95.9, 84.2)
- added TP2: TestPoint, TestPoint:TestPoint_Pad_D1.0mm, B.Cu at (48.2, 26.4)
- added TP3: TestPoint, TestPoint:TestPoint_Pad_D1.0mm, B.Cu at (48.3, 28.9)
- added TP4: TestPoint, TestPoint:TestPoint_Pad_D1.0mm, B.Cu at (48.3, 31.4)
- added TP5: TestPoint, TestPoint:TestPoint_Pad_D1.0mm, B.Cu at (48.3, 36.5)
- added TP6: TestPoint, TestPoint:TestPoint_Pad_D1.0mm, B.Cu at (85.8, 84.1)
- added TP7: TestPoint, TestPoint:TestPoint_Pad_D1.0mm, B.Cu at (88.3, 84.1)
- added TP8: TestPoint, TestPoint:TestPoint_Pad_D1.0mm, B.Cu at (90.8, 84.1)
- added TP9: TestPoint, TestPoint:TestPoint_Pad_D1.0mm, B.Cu at (93.4, 84.1)
- R2: renamed from 10k; footprint Resistor_THT:R_Axial_DIN0309_L9.0mm_D3.2mm_P12.70mm_Horizontal -> Resistor_SMD:R_0603_1608Metric
- R3, R4, R5: footprint Resistor_THT:R_Axial_DIN0309_L9.0mm_D3.2mm_P12.70mm_Horizontal -> Resistor_SMD:R_0603_1608Metric
- moved R5 35.1 mm to (55.7, 74.5), turned to 180 degrees
- moved J2 32.3 mm to (106.5, 72.3)
- moved R4 31.1 mm to (55.7, 77.1), turned to 180 degrees
- moved R3 27.6 mm to (55.7, 79.6), turned to 180 degrees
- moved R2 24.8 mm to (55.7, 82.2), turned to 180 degrees
- moved J6 12.8 mm to (38.0, 42.2)
- moved J1 10.9 mm to (106.5, 39.9)
- renumbered PWR to DP1, XCR to J4, 470 to R1
Connections:
- J6 pad A14: /nOE -> VCC
- J6 pad A16: VCC -> /nCS
- J6 pad A18: /ADR_LOAD -> /nWE
- J6 pad B14: VCC -> /nOE
- J6 pad B16: /nCS -> VCC
- J6 pad B18: /nWE -> /ADR_LOAD
- JCL1 pad 1: /ADR_LOAD -> /nWE
- JCL1 pad 2: /nWE -> /ADR_LOAD
- R1 pad 1: GND -> Net-(R1-Pad1)
Routing:
- net /S0: track 70.2 -> 42.1 mm
- net /S1: track 60.9 -> 38.5 mm
- net /ADR_LOAD: track 31.5 -> 14.7 mm
- net /S2: track 51.4 -> 34.9 mm
- net VCC: track 363.3 -> 347.1 mm
- net /nOE: track 29.9 -> 14.1 mm
- net /W12: track 24.8 -> 10.3 mm
- net /W4: track 34.0 -> 20.5 mm
- net /W2: track 29.8 -> 16.3 mm
- net /W11: track 26.2 -> 12.6 mm
- net /W13: track 25.3 -> 11.8 mm
- net /W3: track 32.5 -> 19.0 mm
- net /W1: track 28.1 -> 14.7 mm
- net /W10: track 27.5 -> 14.6 mm
- net /W5: track 35.0 -> 23.1 mm
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Other:
- board text added: "AL"
- board text added: "CLK"
- board text added: "CS"
- board text added: "D"
- board text added: "DC"
- board text added: "DIN"
- board text added: "EXT"
- board text added: "HDMI"
- board text added: "LED"
- board text added: "PWR"
- board text added: "R"
- board text added: "RES"
- board text added: "SUBSTRATE V0.1"
- board text added: "TOP"
- board text added: "USB-C"
- board text added: "nCS"
- board text added: "nOE"
- board text added: "nWE"
- board text added: "pulldowns"
- board text removed: "SUBSTRATE V0.0"
