File: pcb/v0/v0.kicad_sch (KiCad schematic)
At the start: 22 parts, among them J1 Screw_Terminal_01x02, J2 Screw_Terminal_01x02, J3 Conn_01x08, J4 Conn_01x08, J6 RAM, SW1 SW_DIP_x04

Commit message: substrate fixes
Parts:
- added R6: 470, Resistor_SMD:R_0402_1005Metric, symbol Device:R_US
- added TP1, TP10, TP2, TP3, TP4, TP5, TP6, TP7, TP8, TP9: TestPoint, TestPoint:TestPoint_Pad_D1.0mm, symbol Connector:TestPoint
- R2, R3, R4, R5: footprint Resistor_THT:R_Axial_DIN0309_L9.0mm_D3.2mm_P12.70mm_Horizontal -> Resistor_SMD:R_0603_1608Metric
Connections:
- net ADR_LOAD: now also J6.B18, JCL1.2 (Pin_2), TP2.1; no longer J6.A18, JCL1.1 (Pin_1)
- net GND: now also R6.1; no longer R1.1
- net SCREEN_CLK: now also TP9.1
- net SCREEN_CS: now also TP8.1
- net SCREEN_DC: now also TP7.1
- net SCREEN_DIN: now also TP10.1
- net SCREEN_RES: now also TP6.1
- net VCC: now also J6.A14, J6.B16; no longer J6.A16, J6.B14
- net W0: now also TP5.1
- net nCS: now also J6.A16, TP3.1; no longer J6.B16
- net nOE: now also J6.B14, TP4.1; no longer J6.A14
- net nWE: now also J6.A18, JCL1.1 (Pin_1), TP1.1; no longer J6.B18, JCL1.2 (Pin_2)
- new net: R1.1, R6.2
Other:
- note added: "testpoints"
